File: peripherals/switch_adaptor/switch_adaptor_pcb/switch_adaptor.kicad_pcb (KiCad board)
At the start: 2 copper layers, 25.1 x 23.4 mm, 3 parts, among them J1 PJ320A, J2 PJ320A, J3 PJ320A

Commit message: Updated switch adaptor design
Connections:
- J1 pad 3: Net-(J1-Pad3) -> /Vcc
- J1 pad 5: Net-(J1-Pad5) -> /Vcc
- J2 pad 3: Net-(J2-Pad3) -> /Vcc
- J2 pad 5: Net-(J2-Pad5) -> /Vcc
Other:
- board text added: "Switch Adaptor Ver. 1.1"
- board text added: "https://github.com/ Accessible-AAC"
- board text removed: "Switch Adaptor Ver. 1.0"
Changed lines of the file:
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@@
   (general
     (thickness 1.6)
-    (drawings 19)
+    (drawings 20)
     (tracks 15)
     (zones 0)
     (modules 3)
-    (nets 9)
+    (nets 5)
   )
   (page A4)
@@
   )
   (net 0 "")
-  (net 1 "Net-(J1-Pad5)")
-  (net 2 "Net-(J1-Pad3)")
-  (net 3 "Net-(J2-Pad3)")
-  (net 4 "Net-(J2-Pad5)")
-  (net 5 "Net-(J3-Pad5)")
-  (net 6 /SW1)
-  (net 7 /Vcc)
-  (net 8 /SW2)
+  (net 1 "Net-(J3-Pad5)")
+  (net 2 /SW1)
+  (net 3 /Vcc)
+  (net 4 /SW2)
   (net_class Default "This is the default net class."
     (clearance 0.2)
@@
     (add_net /SW2)
     (add_net /Vcc)
-    (add_net "Net-(J1-Pad3)")
-    (add_net "Net-(J1-Pad5)")
-    (add_net "Net-(J2-Pad3)")
-    (add_net "Net-(J2-Pad5)")
     (add_net "Net-(J3-Pad5)")
   )
@@
     (fp_line (start -3.15 -1.01) (end -3.15 5.09) (layer F.SilkS) (width 0.15))
     (pad 5 thru_hole oval (at 8.15 4.34 270) (size 1.6 2) (drill oval 0.9 1.3) (layers *.Cu *.Mask)
-      (net 5 "Net-(J3-Pad5)"))
+      (net 1 "Net-(J3-Pad5)"))
     (pad 4 thru_hole oval (at 7.05 -0.26 270) (size 1.6 2) (drill oval 0.9 1.3) (layers *.Cu *.Mask)
-      (net 7 /Vcc))
+      (net 3 /Vcc))
     (pad 2 thru_hole oval (at 0.05 -0.26 270) (size 1.6 2) (drill oval 0.9 1.3) (layers *.Cu *.Mask)
-      (net 8 /SW2))
+      (net 4 /SW2))
     (pad "" np_thru_hole circle (at 5.45 2.04 270) (size 0.8 0.8) (drill 0.8) (layers *.Cu *.Mask))
     (pad "" np_thru_hole circle (at -1.55 2.04 270) (size 0.8 0.8) (drill 0.8) (layers *.Cu *.Mask))
     (pad 3 thru_hole oval (at 3.05 -0.26 270) (size 1.6 2) (drill oval 0.9 1.3) (layers *.Cu *.Mask)
-      (net 6 /SW1))
-    (model /home/don/projects/github/Accessible-AAC/Hardware/KiCad_libraries/3D_models/pj320a.wrl
-      (offset (xyz -3.35 -2 0))
-      (scale (xyz 1 1 1))
-      (rotate (xyz 0 0 90))
-    )
+      (net 2 /SW1))
     (model /home/don/kicad/libraries/dbh_kicad_library/3D_models/pj320a/pj320a.wrl
-      (offset (xyz -3.35 -2.1 0))
+      (at (xyz 0 0 0))
       (scale (xyz 1 1 1))
       (rotate (xyz 0 0 0))
@@
     (fp_line (start -3.15 -1.01) (end -3.15 5.09) (layer F.SilkS) (width 0.15))
     (pad 5 thru_hole oval (at 8.15 4.34 90) (size 1.6 2) (drill oval 0.9 1.3) (layers *.Cu *.Mask)
-      (net 4 "Net-(J2-Pad5)"))
+      (net 3 /Vcc))
     (pad 4 thru_hole oval (at 7.05 -0.26 90) (size 1.6 2) (drill oval 0.9 1.3) (layers *.Cu *.Mask)
-      (net 8 /SW2))
+      (net 4 /SW2))
     (pad 2 thru_hole oval (at 0.05 -0.26 90) (size 1.6 2) (drill oval 0.9 1.3) (layers *.Cu *.Mask)
-      (net 7 /Vcc))
+      (net 3 /Vcc))
     (pad "" np_thru_hole circle (at 5.45 2.04 90) (size 0.8 0.8) (drill 0.8) (layers *.Cu *.Mask))
     (pad "" np_thru_hole circle (at -1.55 2.04 90) (size 0.8 0.8) (drill 0.8) (layers *.Cu *.Mask))
     (pad 3 thru_hole oval (at 3.05 -0.26 90) (size 1.6 2) (drill oval 0.9 1.3) (layers *.Cu *.Mask)
-      (net 3 "Net-(J2-Pad3)"))
-    (model /home/don/projects/github/Accessible-AAC/Hardware/KiCad_libraries/3D_models/pj320a.wrl
-      (offset (xyz -3.35 -2 0))
-      (scale (xyz 1 1 1))
-      (rotate (xyz 0 0 90))
-    )
+      (net 3 /Vcc))
     (model /home/don/kicad/libraries/dbh_kicad_library/3D_models/pj320a/pj320a.wrl
-      (offset (xyz -3.35 -2.1 0))
+      (at (xyz 0 0 0))
       (scale (xyz 1 1 1))
       (rotate (xyz 0 0 0))
@@
     (fp_line (start -3.15 -1.01) (end -3.15 5.09) (layer F.SilkS) (width 0.15))
     (pad 5 thru_hole oval (at 8.15 4.34 90) (size 1.6 2) (drill oval 0.9 1.3) (layers *.Cu *.Mask)
-      (net 1 "Net-(J1-Pad5)"))
+      (net 3 /Vcc))
     (pad 4 thru_hole oval (at 7.05 -0.26 90) (size 1.6 2) (drill oval 0.9 1.3) (layers *.Cu *.Mask)
-      (net 6 /SW1))
+      (net 2 /SW1))
     (pad 2 thru_hole oval (at 0.05 -0.26 90) (size 1.6 2) (drill oval 0.9 1.3) (layers *.Cu *.Mask)
-      (net 7 /Vcc))
+      (net 3 /Vcc))
     (pad "" np_thru_hole circle (at 5.45 2.04 90) (size 0.8 0.8) (drill 0.8) (layers *.Cu *.Mask))
     (pad "" np_thru_hole circle (at -1.55 2.04 90) (size 0.8 0.8) (drill 0.8) (layers *.Cu *.Mask))
     (pad 3 thru_hole oval (at 3.05 -0.26 90) (size 1.6 2) (drill oval 0.9 1.3) (layers *.Cu *.Mask)
-      (net 2 "Net-(J1-Pad3)"))
-    (model /home/don/projects/github/Accessible-AAC/Hardware/KiCad_libraries/3D_models/pj320a.wrl
-      (offset (xyz -3.35 -2 0))
-      (scale (xyz 1 1 1))
-      (rotate (xyz 0 0 90))
-    )
+      (net 3 /Vcc))
     (model /home/don/kicad/libraries/dbh_kicad_library/3D_models/pj320a/pj320a.wrl
-      (offset (xyz -3.35 -2.1 0))
+      (at (xyz 0 0 0))
       (scale (xyz 1 1 1))
       (rotate (xyz 0 0 0))
     )
+  )
+  (gr_text "https://github.com/\nAccessible-AAC" (at 136.1186 100.6094) (layer B.SilkS)
+    (effects (font (size 0.8 0.8) (thickness 0.125)) (justify mirror))
   )
   (dimension 12.954 (width 0.15) (layer Dwgs.User)
@@
   (gr_arc (start 141.224 86.868) (end 142.24 86.868) (angle -90) (layer Edge.Cuts) (width 0.05))
   (gr_arc (start 130.302 86.868) (end 130.302 85.852) (angle -90) (layer Edge.Cuts) (width 0.05))
-  (gr_text "Switch Adaptor Ver. 1.0" (at 137.795 97.536) (layer B.SilkS)
+  (gr_text "Switch Adaptor Ver. 1.1" (at 136.8298 97.155) (layer B.SilkS)
     (effects (font (size 0.8 0.8) (thickness 0.125)) (justify mirror))
   )
-  (segment (start 148.334 98.778) (end 148.334 99.828) (width 0.25) (layer F.Cu) (net 6))
-  (segment (start 148.334 96.776) (end 148.334 98.778) (width 0.25) (layer F.Cu) (net 6))
-  (segment (start 148.334 96.594) (end 148.334 96.776) (width 0.25) (layer F.Cu) (net 6))
-  (segment (start 146.812 93.726) (end 148.334 95.248) (width 0.25) (layer F.Cu) (net 6))
-  (segment (start 139.384 87.37) (end 139.384 90.486) (width 0.25) (layer F.Cu) (net 6))
-  (segment (start 138.684 93.726) (end 146.812 93.726) (width 0.25) (layer F.Cu) (net 6))
-  (segment (start 138.176 93.218) (end 138.684 93.726) (width 0.25) (layer F.Cu) (net 6))
-  (segment (start 148.334 95.248) (end 148.334 96.776) (width 0.25) (layer F.Cu) (net 6))
-  (segment (start 139.384 90.486) (end 138.176 91.694) (width 0.25) (layer F.Cu) (net 6))
-  (segment (start 138.176 91.694) (end 138.176 93.218) (width 0.25) (layer F.Cu) (net 6))
-  (segment (start 151.334 100.878) (end 151.334 99.828) (width 0.25) (layer F.Cu) (net 8))
-  (segment (start 150.872 101.34) (end 151.334 100.878) (width 0.25) (layer F.Cu) (net 8))
-  (segment (start 140.634 103.118) (end 139.384 103.118) (width 0.25) (layer F.Cu) (net 8))
-  (segment (start 142.412 101.34) (end 140.634 103.118) (width 0.25) (layer F.Cu) (net 8))
-  (segment (start 150.872 101.34) (end 142.412 101.34) (width 0.25) (layer F.Cu) (net 8))
-  (zone (net 7) (net_name /Vcc) (layer B.Cu) (hatch edge 0.508)
+  (segment (start 148.334 98.778) (end 148.334 99.828) (width 0.25) (layer F.Cu) (net 2))
+  (segment (start 148.334 96.776) (end 148.334 98.778) (width 0.25) (layer F.Cu) (net 2))
+  (segment (start 148.334 96.594) (end 148.334 96.776) (width 0.25) (layer F.Cu) (net 2))
+  (segment (start 146.812 93.726) (end 148.334 95.248) (width 0.25) (layer F.Cu) (net 2))
+  (segment (start 139.384 87.37) (end 139.384 90.486) (width 0.25) (layer F.Cu) (net 2))
+  (segment (start 138.684 93.726) (end 146.812 93.726) (width 0.25) (layer F.Cu) (net 2))
+  (segment (start 138.176 93.218) (end 138.684 93.726) (width 0.25) (layer F.Cu) (net 2))
+  (segment (start 148.334 95.248) (end 148.334 96.776) (width 0.25) (layer F.Cu) (net 2))
+  (segment (start 139.384 90.486) (end 138.176 91.694) (width 0.25) (layer F.Cu) (net 2))
+  (segment (start 138.176 91.694) (end 138.176 93.218) (width 0.25) (layer F.Cu) (net 2))
+  (segment (start 151.334 100.878) (end 151.334 99.828) (width 0.25) (layer F.Cu) (net 4))
+  (segment (start 150.872 101.34) (end 151.334 100.878) (width 0.25) (layer F.Cu) (net 4))
+  (segment (start 140.634 103.118) (end 139.384 103.118) (width 0.25) (layer F.Cu) (net 4))
+  (segment (start 142.412 101.34) (end 140.634 103.118) (width 0.25) (layer F.Cu) (net 4))
+  (segment (start 150.872 101.34) (end 142.412 101.34) (width 0.25) (layer F.Cu) (net 4))
+  (zone (net 3) (net_name /Vcc) (layer B.Cu) (hatch edge 0.508)
     (connect_pads (clearance 0.508))
     (min_thickness 0.254)
